File: sch/converter/v2/power_converter.sch (EAGLE design)
At the start: 22 parts

Commit message: Carrier board
Connections:
- new net SCL: U$1.P$29, U$1.P$30
- new net SDA: U$1.P$27, U$1.P$28
- net EXTVCC: no longer U$1.P$27, U$1.P$28, U$1.P$29, U$1.P$30
- net INTVCC: no longer U$1.P$23, U$1.P$24, U$1.P$25, U$1.P$26
- net PGOOD: now also U$1.P$25, U$1.P$26; no longer U$1.P$21, U$1.P$22
- net RUN: now also U$1.P$23, U$1.P$24; no longer U$1.P$19, U$1.P$20
Changed lines of the file:
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@@
 74439370047</text>
 <text x="217.17" y="20.828" size="2.1844" layer="94">Rev: 2.0</text>
-<wire x1="76.2" y1="38.1" x2="76.2" y2="40.64" width="0.1524" layer="94"/>
-<wire x1="76.2" y1="40.64" x2="85.344" y2="40.64" width="0.1524" layer="94"/>
+<wire x1="60.96" y1="38.1" x2="60.96" y2="40.64" width="0.1524" layer="94"/>
+<wire x1="60.96" y1="40.64" x2="85.344" y2="40.64" width="0.1524" layer="94"/>
 <wire x1="85.344" y1="40.64" x2="93.98" y2="40.64" width="0.1524" layer="94"/>
 <wire x1="93.98" y1="40.64" x2="93.98" y2="38.1" width="0.1524" layer="94"/>
@@
 <label x="76.2" y="137.16" size="1.778" layer="95"/>
 </segment>
-<segment>
-<pinref part="U$1" gate="G$1" pin="P$30"/>
-<wire x1="30.48" y1="33.02" x2="30.48" y2="35.56" width="0.1524" layer="91"/>
-<wire x1="30.48" y1="35.56" x2="33.02" y2="35.56" width="0.1524" layer="91"/>
-<pinref part="U$1" gate="G$1" pin="P$27"/>
-<wire x1="33.02" y1="35.56" x2="38.1" y2="35.56" width="0.1524" layer="91"/>
-<wire x1="38.1" y1="35.56" x2="40.64" y2="35.56" width="0.1524" layer="91"/>
-<wire x1="40.64" y1="35.56" x2="40.64" y2="30.48" width="0.1524" layer="91"/>
-<pinref part="U$1" gate="G$1" pin="P$28"/>
-<wire x1="38.1" y1="33.02" x2="38.1" y2="35.56" width="0.1524" layer="91"/>
-<pinref part="U$1" gate="G$1" pin="P$29"/>
-<wire x1="33.02" y1="30.48" x2="33.02" y2="35.56" width="0.1524" layer="91"/>
-<junction x="33.02" y="35.56"/>
-<junction x="38.1" y="35.56"/>
-<label x="30.734" y="36.322" size="1.778" layer="95"/>
-</segment>
 </net>
 <net name="INTVCC" class="0">
@@
 <label x="40.64" y="96.52" size="1.778" layer="95"/>
 </segment>
+</net>
+<net name="PGOOD" class="0">
+<segment>
+<pinref part="U1" gate="B" pin="PGOOD"/>
+<wire x1="88.9" y1="127" x2="73.66" y2="127" width="0.1524" layer="91"/>
+<label x="76.2" y="127" size="1.778" layer="95"/>
+</segment>
 <segment>
 <pinref part="U$1" gate="G$1" pin="P$26"/>
 <wire x1="45.72" y1="33.02" x2="45.72" y2="35.56" width="0.1524" layer="91"/>
 <wire x1="45.72" y1="35.56" x2="48.26" y2="35.56" width="0.1524" layer="91"/>
-<pinref part="U$1" gate="G$1" pin="P$23"/>
-<wire x1="48.26" y1="35.56" x2="53.34" y2="35.56" width="0.1524" layer="91"/>
-<wire x1="53.34" y1="35.56" x2="55.88" y2="35.56" width="0.1524" layer="91"/>
-<wire x1="55.88" y1="35.56" x2="55.88" y2="30.48" width="0.1524" layer="91"/>
-<pinref part="U$1" gate="G$1" pin="P$24"/>
-<wire x1="53.34" y1="33.02" x2="53.34" y2="35.56" width="0.1524" layer="91"/>
 <pinref part="U$1" gate="G$1" pin="P$25"/>
 <wire x1="48.26" y1="30.48" x2="48.26" y2="35.56" width="0.1524" layer="91"/>
-<junction x="48.26" y="35.56"/>
-<junction x="53.34" y="35.56"/>
-<label x="45.72" y="36.322" size="1.778" layer="95"/>
-</segment>
-</net>
-<net name="PGOOD" class="0">
-<segment>
-<pinref part="U1" gate="B" pin="PGOOD"/>
-<wire x1="88.9" y1="127" x2="73.66" y2="127" width="0.1524" layer="91"/>
-<label x="76.2" y="127" size="1.778" layer="95"/>
-</segment>
-<segment>
-<pinref part="U$1" gate="G$1" pin="P$22"/>
-<wire x1="60.96" y1="33.02" x2="60.96" y2="35.56" width="0.1524" layer="91"/>
-<wire x1="60.96" y1="35.56" x2="63.5" y2="35.56" width="0.1524" layer="91"/>
-<pinref part="U$1" gate="G$1" pin="P$21"/>
-<wire x1="63.5" y1="35.56" x2="63.5" y2="30.48" width="0.1524" layer="91"/>
-<label x="60.452" y="33.02" size="1.778" layer="95" rot="R90"/>
+<label x="45.212" y="33.02" size="1.778" layer="95" rot="R90"/>
 </segment>
 </net>
@@
 </segment>
 <segment>
-<pinref part="U$1" gate="G$1" pin="P$20"/>
-<wire x1="68.58" y1="33.02" x2="68.58" y2="35.56" width="0.1524" layer="91"/>
-<wire x1="68.58" y1="35.56" x2="71.12" y2="35.56" width="0.1524" layer="91"/>
-<pinref part="U$1" gate="G$1" pin="P$19"/>
-<wire x1="71.12" y1="35.56" x2="71.12" y2="30.48" width="0.1524" layer="91"/>
-<label x="68.072" y="33.02" size="1.778" layer="95" rot="R90"/>
-</segment>
-<segment>
 <wire x1="43.18" y1="129.54" x2="43.18" y2="124.46" width="0.1524" layer="91"/>
 <wire x1="33.02" y1="129.54" x2="43.18" y2="129.54" width="0.1524" layer="91"/>
@@
 <pinref part="R3" gate="G$1" pin="2"/>
 <wire x1="33.02" y1="129.54" x2="33.02" y2="124.46" width="0.1524" layer="91"/>
+</segment>
+<segment>
+<pinref part="U$1" gate="G$1" pin="P$23"/>
+<wire x1="53.34" y1="35.56" x2="55.88" y2="35.56" width="0.1524" layer="91"/>
+<wire x1="55.88" y1="35.56" x2="55.88" y2="30.48" width="0.1524" layer="91"/>
+<pinref part="U$1" gate="G$1" pin="P$24"/>
+<wire x1="53.34" y1="33.02" x2="53.34" y2="35.56" width="0.1524" layer="91"/>
+<label x="52.832" y="33.02" size="1.778" layer="95" rot="R90"/>
 </segment>
 </net>
@@
 </segment>
 </net>
+<net name="SCL" class="0">
+<segment>
+<pinref part="U$1" gate="G$1" pin="P$30"/>
+<wire x1="30.48" y1="33.02" x2="30.48" y2="35.56" width="0.1524" layer="91"/>
+<wire x1="30.48" y1="35.56" x2="33.02" y2="35.56" width="0.1524" layer="91"/>
+<pinref part="U$1" gate="G$1" pin="P$29"/>
+<wire x1="33.02" y1="30.48" x2="33.02" y2="35.56" width="0.1524" layer="91"/>
+<label x="30.226" y="35.814" size="1.778" layer="95" rot="R90"/>
+</segment>
+</net>
+<net name="SDA" class="0">
+<segment>
+<pinref part="U$1" gate="G$1" pin="P$27"/>
+<wire x1="38.1" y1="35.56" x2="40.64" y2="35.56" width="0.1524" layer="91"/>
+<wire x1="40.64" y1="35.56" x2="40.64" y2="30.48" width="0.1524" layer="91"/>
+<pinref part="U$1" gate="G$1" pin="P$28"/>
+<wire x1="38.1" y1="33.02" x2="38.1" y2="35.56" width="0.1524" layer="91"/>
+<label x="37.846" y="35.814" size="1.778" layer="95" rot="R90"/>
+</segment>
+</net>

Commit message: Added carrier BOM; Chaned carrier MOSFETs
Changed lines of the file:
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@@
 <segment>
 <pinref part="U1" gate="B" pin="PLLFLTR"/>
-<wire x1="88.9" y1="96.52" x2="73.66" y2="96.52" width="0.1524" layer="91"/>
+<wire x1="88.9" y1="96.52" x2="66.04" y2="96.52" width="0.1524" layer="91"/>
 <label x="76.2" y="96.52" size="1.778" layer="95"/>
-</segment>
-<segment>
 <pinref part="R6" gate="G$1" pin="1"/>
 <wire x1="63.5" y1="96.52" x2="66.04" y2="96.52" width="0.1524" layer="91"/>
 <pinref part="R9" gate="G$1" pin="1"/>
 <wire x1="66.04" y1="96.52" x2="66.04" y2="91.44" width="0.1524" layer="91"/>
-<wire x1="66.04" y1="96.52" x2="73.66" y2="96.52" width="0.1524" layer="91"/>
 <junction x="66.04" y="96.52"/>
 </segment>

Commit message: Updated CAM files
Changed lines of the file:
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@@
 <?xml version="1.0" encoding="utf-8"?>
 <!DOCTYPE eagle SYSTEM "eagle.dtd">
-<eagle version="9.1.3">
+<eagle version="9.2.1">
 <drawing>
 <settings>
@@
 <layer number="98" name="Guide" color="6" fill="1" visible="yes" active="yes"/>
 <layer number="99" name="SpiceOrder" color="5" fill="1" visible="yes" active="yes"/>
+<layer number="100" name="Parts" color="7" fill="1" visible="yes" active="yes"/>
+<layer number="250" name="Descript" color="7" fill="1" visible="yes" active="yes"/>
+<layer number="251" name="SMDround" color="7" fill="1" visible="yes" active="yes"/>
 </layers>
 <schematic xreflabel="%F%N/%S.%C%R" xrefpart="/%S.%C%R">
@@
 </plain>
 <instances>
-<instance part="FRAME1" gate="G$1" x="0" y="0"/>
-<instance part="U1" gate="B" x="93.98" y="137.16"/>
-<instance part="L1" gate="G$1" x="157.48" y="132.08" rot="R90"/>
-<instance part="R5" gate="G$1" x="154.94" y="106.68"/>
-<instance part="GND7" gate="1" x="147.32" y="86.36"/>
-<instance part="C8" gate="G$1" x="167.64" y="116.84"/>
-<instance part="C9" gate="G$1" x="175.26" y="116.84"/>
-<instance part="GND5" gate="1" x="167.64" y="104.14"/>
-<instance part="GND1" gate="1" x="177.8" y="132.08"/>
-<instance part="R7" gate="G$1" x="195.58" y="91.44" rot="R180"/>
-<instance part="GND8" gate="1" x="215.9" y="86.36"/>
-<instance part="R6" gate="G$1" x="58.42" y="96.52" rot="R180"/>
-<instance part="R9" gate="G$1" x="66.04" y="86.36" rot="R270"/>
-<instance part="C16" gate="G$1" x="63.5" y="106.68" rot="R90"/>
-<instance part="D1" gate="G$1" x="43.18" y="116.84" rot="R90"/>
-<instance part="GND3" gate="1" x="43.18" y="109.22"/>
-<instance part="R1" gate="G$1" x="43.18" y="139.7" rot="R90"/>
-<instance part="GND9" gate="1" x="66.04" y="76.2"/>
-<instance part="GND6" gate="1" x="86.36" y="86.36"/>
-<instance part="GND4" gate="1" x="55.88" y="106.68" rot="R270"/>
-<instance part="R3" gate="G$1" x="33.02" y="119.38" rot="R90"/>
-<instance part="GND2" gate="1" x="33.02" y="109.22"/>
-<instance part="C7" gate="G$1" x="195.58" y="144.78"/>
-<instance part="R8" gate="G$1" x="208.28" y="91.44" rot="R180"/>
-<instance part="R4" gate="G$1" x="154.94" y="114.3"/>
-<instance part="C14" gate="G$1" x="193.04" y="116.84"/>
-<instance part="U$1" gate="G$1" x="12.7" y="15.24"/>
-<instance part="C2" gate="G$1" x="182.88" y="116.84"/>
-<instance part="C3" gate="G$1" x="203.2" y="116.84"/>
-<instance part="C4" gate="G$1" x="177.8" y="144.78"/>
-<instance part="C5" gate="G$1" x="185.42" y="144.78"/>
-<instance part="F1" gate="G$1" x="205.74" y="149.86"/>
+<instance part="FRAME1" gate="G$1" x="0" y="0" smashed="yes">
+<attribute name="DRAWING_NAME" x="217.17" y="15.24" size="2.54" layer="94"/>
+<attribute name="LAST_DATE_TIME" x="217.17" y="10.16" size="2.286" layer="94"/>
+<attribute name="SHEET" x="230.505" y="5.08" size="2.54" layer="94"/>
+</instance>
+<instance part="U1" gate="B" x="93.98" y="137.16" smashed="yes">
+<attribute name="NAME" x="115.57" y="88.9" size="2.54" layer="94" ratio="6" align="bottom-center"/>
+</instance>
+<instance part="L1" gate="G$1" x="157.48" y="132.08" smashed="yes" rot="R90">
+<attribute name="NAME" x="162.56" y="130.81" size="1.778" layer="95" rot="R180"/>
+<attribute name="VALUE" x="162.56" y="135.89" size="1.778" layer="96" rot="R180"/>
+</instance>
+<instance part="R5" gate="G$1" x="154.94" y="106.68" smashed="yes">
+<attribute name="NAME" x="151.13" y="108.1786" size="1.778" layer="95"/>
+<attribute name="VALUE" x="151.13" y="103.378" size="1.778" layer="96"/>
+</instance>
+<instance part="GND7" gate="1" x="147.32" y="86.36" smashed="yes">
+<attribute name="VALUE" x="144.78" y="83.82" size="1.778" layer="96"/>
+</instance>
+<instance part="C8" gate="G$1" x="167.64" y="116.84" smashed="yes">
+<attribute name="NAME" x="169.164" y="117.221" size="1.778" layer="95"/>
+<attribute name="VALUE" x="169.164" y="112.141" size="1.778" layer="96"/>
+</instance>
+<instance part="C9" gate="G$1" x="175.26" y="116.84" smashed="yes">
+<attribute name="NAME" x="176.784" y="117.221" size="1.778" layer="95"/>
+<attribute name="VALUE" x="176.784" y="112.141" size="1.778" layer="96"/>
+</instance>
+<instance part="GND5" gate="1" x="167.64" y="104.14" smashed="yes">
+<attribute name="VALUE" x="165.1" y="101.6" size="1.778" layer="96"/>
+</instance>
+<instance part="GND1" gate="1" x="177.8" y="132.08" smashed="yes">
+<attribute name="VALUE" x="175.26" y="129.54" size="1.778" layer="96"/>
+</instance>
+<instance part="R7" gate="G$1" x="195.58" y="91.44" smashed="yes" rot="R180">
+<attribute name="NAME" x="199.39" y="89.9414" size="1.778" layer="95" rot="R180"/>
+<attribute name="VALUE" x="199.39" y="94.742" size="1.778" layer="96" rot="R180"/>
+</instance>
+<instance part="GND8" gate="1" x="215.9" y="86.36" smashed="yes">
+<attribute name="VALUE" x="213.36" y="83.82" size="1.778" layer="96"/>
+</instance>
+<instance part="R6" gate="G$1" x="58.42" y="96.52" smashed="yes" rot="R180">
+<attribute name="NAME" x="62.23" y="95.0214" size="1.778" layer="95" rot="R180"/>
+<attribute name="VALUE" x="62.23" y="99.822" size="1.778" layer="96" rot="R180"/>
+</instance>
+<instance part="R9" gate="G$1" x="66.04" y="86.36" smashed="yes" rot="R270">
+<attribute name="NAME" x="67.5386" y="90.17" size="1.778" layer="95" rot="R270"/>
+<attribute name="VALUE" x="62.738" y="90.17" size="1.778" layer="96" rot="R270"/>
+</instance>
+<instance part="C16" gate="G$1" x="63.5" y="106.68" smashed="yes" rot="R90">
+<attribute name="NAME" x="63.119" y="108.204" size="1.778" layer="95" rot="R90"/>
+<attribute name="VALUE" x="68.199" y="108.204" size="1.778" layer="96" rot="R90"/>
+</instance>
+<instance part="D1" gate="G$1" x="43.18" y="116.84" smashed="yes" rot="R90">
+<attribute name="NAME" x="41.275" y="115.062" size="1.778" layer="95" rot="R90"/>
+<attribute name="VALUE" x="46.609" y="115.062" size="1.778" layer="96" rot="R90"/>
+</instance>
+<instance part="GND3" gate="1" x="43.18" y="109.22" smashed="yes">
+<attribute name="VALUE" x="40.64" y="106.68" size="1.778" layer="96"/>
+</instance>
+<instance part="R1" gate="G$1" x="43.18" y="139.7" smashed="yes" rot="R90">
+<attribute name="NAME" x="41.6814" y="135.89" size="1.778" layer="95" rot="R90"/>
+<attribute name="VALUE" x="46.482" y="135.89" size="1.778" layer="96" rot="R90"/>
+</instance>
+<instance part="GND9" gate="1" x="66.04" y="76.2" smashed="yes">
+<attribute name="VALUE" x="63.5" y="73.66" size="1.778" layer="96"/>
+</instance>
+<instance part="GND6" gate="1" x="86.36" y="86.36" smashed="yes">
+<attribute name="VALUE" x="83.82" y="83.82" size="1.778" layer="96"/>
+</instance>
+<instance part="GND4" gate="1" x="55.88" y="106.68" smashed="yes" rot="R270">
+<attribute name="VALUE" x="53.34" y="109.22" size="1.778" layer="96" rot="R270"/>
+</instance>
+<instance part="R3" gate="G$1" x="33.02" y="119.38" smashed="yes" rot="R90">
+<attribute name="NAME" x="31.5214" y="115.57" size="1.778" layer="95" rot="R90"/>
+<attribute name="VALUE" x="36.322" y="115.57" size="1.778" layer="96" rot="R90"/>
+</instance>
+<instance part="GND2" gate="1" x="33.02" y="109.22" smashed="yes">
+<attribute name="VALUE" x="30.48" y="106.68" size="1.778" layer="96"/>
+</instance>
+<instance part="C7" gate="G$1" x="195.58" y="144.78" smashed="yes">
+<attribute name="NAME" x="196.596" y="145.415" size="1.778" layer="95"/>
+<attribute name="VALUE" x="196.596" y="140.589" size="1.778" layer="96"/>
+</instance>
+<instance part="R8" gate="G$1" x="208.28" y="91.44" smashed="yes" rot="R180">
+<attribute name="NAME" x="212.09" y="89.9414" size="1.778" layer="95" rot="R180"/>
+<attribute name="VALUE" x="212.09" y="94.742" size="1.778" layer="96" rot="R180"/>
+</instance>
+<instance part="R4" gate="G$1" x="154.94" y="114.3" smashed="yes">
+<attribute name="NAME" x="151.13" y="115.7986" size="1.778" layer="95"/>
+<attribute name="VALUE" x="151.13" y="110.998" size="1.778" layer="96"/>
+</instance>
+<instance part="C14" gate="G$1" x="193.04" y="116.84" smashed="yes">
+<attribute name="NAME" x="194.056" y="117.475" size="1.778" layer="95"/>
+<attribute name="VALUE" x="194.056" y="112.649" size="1.778" layer="96"/>
+</instance>
+<instance part="U$1" gate="G$1" x="12.7" y="15.24" smashed="yes"/>
+<instance part="C2" gate="G$1" x="182.88" y="116.84" smashed="yes">
+<attribute name="NAME" x="184.404" y="117.221" size="1.778" layer="95"/>
+<attribute name="VALUE" x="184.404" y="112.141" size="1.778" layer="96"/>
+</instance>
+<instance part="C3" gate="G$1" x="203.2" y="116.84" smashed="yes">
+<attribute name="NAME" x="204.216" y="117.475" size="1.778" layer="95"/>
+<attribute name="VALUE" x="204.216" y="112.649" size="1.778" layer="96"/>
+</instance>
+<instance part="C4" gate="G$1" x="177.8" y="144.78" smashed="yes">
+<attribute name="NAME" x="179.324" y="145.161" size="1.778" layer="95"/>
+<attribute name="VALUE" x="179.324" y="140.081" size="1.778" layer="96"/>
+</instance>
+<instance part="C5" gate="G$1" x="185.42" y="144.78" smashed="yes">
+<attribute name="NAME" x="186.944" y="145.161" size="1.778" layer="95"/>
+<attribute name="VALUE" x="186.944" y="140.081" size="1.778" layer="96"/>
+</instance>
+<instance part="F1" gate="G$1" x="205.74" y="149.86" smashed="yes">
+<attribute name="NAME" x="201.93" y="151.257" size="1.778" layer="95"/>
+<attribute name="VALUE" x="201.93" y="146.939" size="1.778" layer="96"/>
+</instance>
 </instances>
 <busses>
