File: sch/carrier/carrier_board.brd (EAGLE design)
At the start: 100 x 100 mm, 93 parts, among them CON1 SM03B-GHS-TB, CON2 SM03B-GHS-TB, Q1 SI7145, Q2 SI7145, Q3 SI7145, Q4 SIJ438DP, Q5 SIJ438DP, Q6 SIJ438DP, Q7 SIJ438DP, U1 LTV-355T, U10 LTC4418, U11 TEENSY_3.1_BASIC_2, U12 MCP2562, U3 LTV-355T, U4 LTV-355T, U6 LTV-355T, U7 LTV-355T, U9 LTV-355T

Commit message: Updated CAM files
Routing:
- net V1: track 43.6 -> 45.0 mm
Changed lines of the file:
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@@
 <layer number="28" name="bValues" color="7" fill="1" visible="no" active="yes"/>
 <layer number="29" name="tStop" color="7" fill="3" visible="yes" active="yes"/>
-<layer number="30" name="bStop" color="7" fill="6" visible="yes" active="yes"/>
+<layer number="30" name="bStop" color="7" fill="6" visible="no" active="yes"/>
 <layer number="31" name="tCream" color="7" fill="4" visible="yes" active="yes"/>
 <layer number="32" name="bCream" color="7" fill="5" visible="yes" active="yes"/>
@@
 <wire x1="114.155" y1="124.96" x2="113.7067125" y2="124.96" width="0.1524" layer="1"/>
 <wire x1="113.4514" y1="125.2153125" x2="113.4514" y2="127.8486" width="0.1524" layer="1"/>
-<wire x1="112.649" y1="136.144" x2="112.903" y2="136.398" width="0.1524" layer="1"/>
-<wire x1="112.903" y1="136.398" x2="127.382" y2="136.398" width="0.1524" layer="1"/>
-<wire x1="127.382" y1="136.398" x2="130.81" y2="135.0344" width="0.1524" layer="1"/>
+<wire x1="112.903" y1="136.398" x2="112.649" y2="136.144" width="0.1524" layer="1"/>
 <wire x1="113.4514" y1="127.8486" x2="112.649" y2="128.651" width="0.1524" layer="1"/>
 <wire x1="112.649" y1="128.651" x2="112.649" y2="136.144" width="0.1524" layer="1"/>
@@
 <wire x1="136.7282" y1="131.699" x2="135.0772" y2="133.35" width="1.27" layer="16"/>
 <wire x1="135.0772" y1="133.35" x2="131.145" y2="133.35" width="1.27" layer="16"/>
+<wire x1="130.81" y1="132.94" x2="128.495" y2="135.255" width="0.1524" layer="1"/>
+<wire x1="128.495" y1="135.255" x2="128.016" y2="135.255" width="0.1524" layer="1"/>
+<wire x1="128.016" y1="135.255" x2="127.635" y2="135.636" width="0.1524" layer="1"/>
+<wire x1="127.635" y1="135.636" x2="127.635" y2="136.017" width="0.1524" layer="1"/>
+<wire x1="127.635" y1="136.017" x2="127.254" y2="136.398" width="0.1524" layer="1"/>
+<wire x1="127.254" y1="136.398" x2="112.903" y2="136.398" width="0.1524" layer="1"/>
 </signal>
 <signal name="V2">

Commit message: Revision 1.2
Parts:
- added C10, C9: 100n, rcl:C0603
- added Q8: BSS123, transistor-small-signal:SOT23
- added R35, R36: 1k, rcl:R0603
- C7, C8: value 10u -> 100n
- D4, D5: value 5.0SMDJ40CA -> SMBJ30CA; device 5.0SMDJ40CA:DIOM794X590X262L114X305N -> LTM4607:DO214AA
- Q1, Q2, Q3: value SI7145 -> SQJ407EP
- Q4, Q5, Q6, Q7: value SIJ438DP -> SI7145DP; device LTM4607:POWERPAK_SO8L_SINGLE -> LTM4607:SO-8-POWERPAK
- R20, R23: value 234k -> 210k
- R21, R24: value 124k -> 150k
- R25, R27: device rcl:R0402 -> rcl:R0603
- U13: value (none) -> VX7805-500; device LTM4607:SRH05 -> LTM4607:0.1"_LINEAR_REGULATOR_REPLACEMENT
- X1, X3, X5: device LTM4607:282834-8 -> LTM4607:284391-6
- moved D5 2.54 mm to (130.2, 133.3)
- moved D4 2.54 mm to (108.6, 133.3)
- moved R25 1.42 mm to (86.4, 135.9), turned to 90 degrees
- moved R27 1.42 mm to (83.8, 135.9), turned to 90 degrees
- moved Q1 0.51 mm to (65.2, 108.0)
- moved Q2 0.51 mm to (65.2, 86.4)
- moved Q3 0.51 mm to (65.2, 64.8)
- turned X1 to 270 degrees
- turned X3 to 270 degrees
- turned X5 to 270 degrees
Connections:
- new net G1_DRIVER: R36.1, U10.13
- new net G2_DRIVER: R35.1, U10.11
- new net N$10: Q8.1, U11.2
- net +5V: now also R25.1, R27.1; no longer R25.2, R27.2
- net /VALID1: now also R25.2, U11.14/A0; no longer R25.1, U11.13
- net /VALID2: now also R27.2, U11.15/A1; no longer R27.1, U11.14/A0
- net G1: now also C10.2, Q6.4, Q7.4, R36.2; no longer Q6.P$4, Q7.P$4, U10.13
- net G2: now also C9.2, Q4.4, Q5.4, R35.2; no longer Q4.P$4, Q5.P$4, U10.11
- net GND: now also D4.A, D5.A, Q8.2, X1.P$1, X1.P$2, X1.P$3, X3.P$1, X3.P$2, X3.P$3, X5.P$1, X5.P$2, X5.P$3; no longer D4.2, D5.2, X1.P$5, X1.P$6, X1.P$7, X1.P$8, X3.P$5, X3.P$6, X3.P$7, X3.P$8, X5.P$5, X5.P$6, X5.P$7, X5.P$8
- net INTVCC: now also U10.18, U10.19
- net KILL_SWITCH_C: now also Q8.3
- net V1: now also D5.C, Q6.5, Q6.6, Q6.7, Q6.8, Q6.P$1; no longer D5.1, Q6.P$5, Q6.P$6, Q6.P$7, Q6.P$8
- net V2: now also D4.C, Q4.5, Q4.6, Q4.7, Q4.8, Q4.P$1; no longer D4.1, Q4.P$5, Q4.P$6, Q4.P$7, Q4.P$8
- net VIN: now also C10.1, C9.1, Q5.5, Q5.6, Q5.7, Q5.8, Q5.P$1, Q7.5, Q7.6, Q7.7, Q7.8, Q7.P$1; no longer Q5.P$5, Q5.P$6, Q5.P$7, Q5.P$8, Q7.P$5, Q7.P$6, Q7.P$7, Q7.P$8
- net VOUT1: now also X1.P$5, X1.P$6; no longer X1.P$1, X1.P$2
- net VOUT2: now also X3.P$5, X3.P$6; no longer X3.P$1, X3.P$2
- net VOUT3: now also X5.P$5, X5.P$6; no longer X5.P$1, X5.P$2
- net VOUT_SWITCHED1: no longer X1.P$3
- net VOUT_SWITCHED2: no longer X3.P$3
- net VOUT_SWITCHED3: no longer X5.P$3
- net VS1: now also Q6.1, Q6.2, Q6.3, Q7.1, Q7.2, Q7.3; no longer Q6.P$1, Q6.P$2, Q6.P$3, Q7.P$1, Q7.P$2, Q7.P$3
- net VS2: now also Q4.1, Q4.2, Q4.3, Q5.1, Q5.2, Q5.3; no longer Q4.P$1, Q4.P$2, Q4.P$3, Q5.P$1, Q5.P$2, Q5.P$3
Routing:
- net KILL_SWITCH_C: track 108.4 -> 142.7 mm
- net INTVCC: track 1.78 -> 31.3 mm, vias 0 -> 2
- net G1: track 29.8 -> 12.0 mm, vias 0 -> 1
- net G1_DRIVER: track 0.00 -> 17.8 mm, vias 0 -> 1
- net /VALID1: track 53.2 -> 61.9 mm
- net /VALID2: track 58.5 -> 66.5 mm
- net G2_DRIVER: track 0.00 -> 7.66 mm, vias 0 -> 1
- net VIN: track 49.6 -> 52.6 mm, vias 2 -> 4
- net N$10: track 0.00 -> 2.77 mm
- net VOUT3: track 11.1 -> 13.9 mm
- net VOUT1: track 11.1 -> 13.9 mm
- net VOUT2: track 11.1 -> 13.9 mm
- net +5V: track 295.3 -> 297.7 mm
- net G2: track 15.2 -> 13.5 mm, vias 0 -> 1
- net V2: track 30.3 -> 28.7 mm
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Other:
- board text added: "ALAIN L. 2018-11"
- board text added: "INPUT: 12.5-30V"
- board text added: "NOTES: 1. Solder board in following order: 1.1 Reflow solder top surface mounted components except edge connectors 1.2 Hand solder bottom components 1.3 Hand solder remaining top components 1.3.1 Solder edge connectors first 2. Use LP MINI 891 fuses for F1 through F5 3. 2oz copper suggested, but not required"
- board text added: "REV. 1.2"
- board text removed: "ALAIN L. 2018-10"
- board text removed: "INPUT: 12.5-36V"
- board text removed: "NOTES: 1. Solder board in following order: 1.1 Reflow solder top surface mounted components 1.2 Hand solder bottom components 1.3 Hand solder remaining top components 2. Use LP MINI 891 fuses for F1 through F5 3. 2oz copper recommended"

Commit message: Carrier rev. 1.3
Parts:
- added D6, D7: (no value), LTM4607:CHIPLED_0603
- added R37: 0, rcl:R0402
- R35, R36: value 1k -> 2k
- moved C4 0.92 mm to (111.6, 121.2), turned to 90 degrees
Connections:
- net G1: now also D7.C
- net G1_DRIVER: now also D7.A
- net G2: now also D6.C
- net G2_DRIVER: now also D6.A
- net INTVCC: now also R37.1
- net TMR: now also R37.2
Routing:
- net G2_DRIVER: track 7.66 -> 9.22 mm
- net G2: track 13.5 -> 15.1 mm
- net G1_DRIVER: track 17.8 -> 19.3 mm
- net G1: track 12.0 -> 13.6 mm
- net TMR: track 3.63 -> 5.16 mm
Other:
- board text added: "ALAIN L. 2018-12"
- board text added: "REV. 1.3"
- board text removed: "ALAIN L. 2018-11"
- board text removed: "REV. 1.2"
