File: sch/carrier/carrier_board.brd (EAGLE design)
At the start: 100 x 100 mm, 101 parts, among them CON1 SM03B-GHS-TB, CON2 SM03B-GHS-TB, Q1 SQJ407EP, Q2 SQJ407EP, Q3 SQJ407EP, Q4 SI7145DP, Q5 SI7145DP, Q6 SI7145DP, Q7 SI7145DP, Q8 BSS123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

Commit message: Carrier rev. 1.4
Parts:
- added D8: MBRS2040LT3G, diode:SMB
- added R38: 50k, rcl:R0603
- added R39: 5k, rcl:R0603
- added U$7: (no value), oshw:OSHW_5MM
- moved U13 1.27 mm to (92.7, 125.7)
Connections:
- new net N$11: D8.C, U13.1
- new net V1_ANALOG_IN: R38.1, R39.2, U11.17/A3
- net GND: now also R39.1
- net N$1: now also D8.A, R38.2; no longer U13.1
Routing:
- net N$1: track 8.95 -> 27.4 mm
- net V1_ANALOG_IN: track 0.00 -> 12.0 mm
- net N$11: track 0.00 -> 7.62 mm
Other:
- board text added: "ALAIN L. 2019-10"
- board text added: "REV. 1.4"
- board text removed: "ALAIN L. 2018-12"
- board text removed: "REV. 1.3"
